File: PCB/Shematich_v1.brd (EAGLE design)
At the start: 100 x 80 mm, 8 parts, among them U1 EK-TM4C123GXL, U2 4N25, X1 HD44780LCD-1602, X2 22-23-2081, X3 22-23-2031

Commit message: shematic 3
Parts:
- added U$2: (no value), keypad_4x4_raw:KEYPAD4X4
Changed lines of the file:
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@@
 <attribute name="VALUE" x="-110.8456" y="-15.7226" size="0.9906" layer="27" ratio="10"/>
+</element>
+<element name="U$2" library="keypad_4x4_raw" package="KEYPAD4X4" value="" x="-179.07" y="-8.89" smashed="yes">
+<attribute name="NAME" x="-170.3362" y="-11.3612" size="1.27" layer="25" ratio="10"/>
+<attribute name="VALUE" x="-128.1" y="-11.555" size="1.27" layer="27"/>
 </element>
 </elements>

Commit message: final schematic
Parts:
- removed X2: 22-23-2081, con-molex:22-23-2081
- added R2, R3, R4, R5: 320, rcl:0204/7
Connections:
- removed net +3.3V: U1.J1_1
- removed net N$11 (its old number): R1.2, U1.J1_6
- removed net SCL: U$1.P$1
- removed net SDA: U$1.P$6
- new net N$1: R1.2, U1.J4_3
- new net N$13: R2.2, U$2.4, U1.J3_6
- new net N$14: R4.2, U$2.2, U1.J3_4
- new net N$16: U$2.5, U1.J1_7
- new net N$17: U$2.6, U1.J1_2
- new net N$18: U$2.7, U1.J2_7
- new net N$19: U$2.8, U1.J2_6
- new net N$20: R5.2, U$2.1, U1.J3_3
- new net N$3: R3.2, U$2.3, U1.J3_5
- new net VDD: X1.2
- net GND: now also R2.1, R3.1, R4.1, R5.1
- net N$4: now also U$1.P$1, U1.J1_6; no longer U$1.P$5
- net N$5: now also U$1.P$6, U1.J1_5; no longer U$1.P$3
- net UART_RX: now also U1.J1_4
- net UART_TX: now also U1.J1_3
- net VCC: now also U1.J1_1
Changed lines of the file:
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@@
 </element>
 <element name="X1" library="adafruit" library_urn="urn:adsk.eagle:library:420" package="LCD1602" package3d_urn="urn:adsk.eagle:package:6240760/1" value="HD44780LCD-1602" x="-93.98" y="72.39" smashed="yes"/>
-<element name="X2" library="con-molex" library_urn="urn:adsk.eagle:library:165" package="22-23-2081" package3d_urn="urn:adsk.eagle:package:8078639/1" value="22-23-2081" x="-83.82" y="-6.35" smashed="yes">
-<attribute name="MF" value="MOLEX" x="-83.82" y="-6.35" size="1.778" layer="27" display="off"/>
-<attribute name="MPN" value="22-23-2081" x="-83.82" y="-6.35" size="1.778" layer="27" display="off"/>
-<attribute name="NAME" x="-93.98" y="-2.54" size="1.016" layer="25" ratio="10"/>
-<attribute name="OC_FARNELL" value="1756826" x="-83.82" y="-6.35" size="1.778" layer="27" display="off"/>
-<attribute name="OC_NEWARK" value="01C7592" x="-83.82" y="-6.35" size="1.778" layer="27" display="off"/>
-<attribute name="POPULARITY" value="0" x="-83.82" y="-6.35" size="1.778" layer="27" display="off"/>
-<attribute name="VALUE" x="-93.98" y="-11.43" size="1.016" layer="27" ratio="10"/>
-</element>
 <element name="X3" library="con-molex" library_urn="urn:adsk.eagle:library:165" package="22-23-2031" package3d_urn="urn:adsk.eagle:package:8078634/1" value="22-23-2031" x="-99.06" y="-6.35" smashed="yes">
 <attribute name="MF" value="MOLEX" x="-99.06" y="-6.35" size="1.778" layer="27" display="off"/>
@@
 <attribute name="VALUE" x="-128.1" y="-11.555" size="1.27" layer="27"/>
 </element>
+<element name="R2" library="rcl" library_urn="urn:adsk.eagle:library:334" package="0204/7" package3d_urn="urn:adsk.eagle:package:23498/2" value="320" x="-175.26" y="-20.32" smashed="yes">
+<attribute name="NAME" x="-177.8" y="-19.0246" size="0.9906" layer="25" ratio="10"/>
+<attribute name="POPULARITY" value="48" x="-175.26" y="-20.32" size="1.778" layer="27" display="off"/>
+<attribute name="SPICEPREFIX" value="R" x="-175.26" y="-20.32" size="1.778" layer="27" display="off"/>
+<attribute name="VALUE" x="-176.8856" y="-20.8026" size="0.9906" layer="27" ratio="10"/>
+</element>
+<element name="R3" library="rcl" library_urn="urn:adsk.eagle:library:334" package="0204/7" package3d_urn="urn:adsk.eagle:package:23498/2" value="320" x="-175.26" y="-25.4" smashed="yes">
+<attribute name="NAME" x="-177.8" y="-24.1046" size="0.9906" layer="25" ratio="10"/>
+<attribute name="POPULARITY" value="48" x="-175.26" y="-25.4" size="1.778" layer="27" display="off"/>
+<attribute name="SPICEPREFIX" value="R" x="-175.26" y="-25.4" size="1.778" layer="27" display="off"/>
+<attribute name="VALUE" x="-176.8856" y="-25.8826" size="0.9906" layer="27" ratio="10"/>
+</element>
+<element name="R4" library="rcl" library_urn="urn:adsk.eagle:library:334" package="0204/7" package3d_urn="urn:adsk.eagle:package:23498/2" value="320" x="-175.26" y="-30.48" smashed="yes">
+<attribute name="NAME" x="-177.8" y="-29.1846" size="0.9906" layer="25" ratio="10"/>
+<attribute name="POPULARITY" value="48" x="-175.26" y="-30.48" size="1.778" layer="27" display="off"/>
+<attribute name="SPICEPREFIX" value="R" x="-175.26" y="-30.48" size="1.778" layer="27" display="off"/>
+<attribute name="VALUE" x="-176.8856" y="-30.9626" size="0.9906" layer="27" ratio="10"/>
+</element>
+<element name="R5" library="rcl" library_urn="urn:adsk.eagle:library:334" package="0204/7" package3d_urn="urn:adsk.eagle:package:23498/2" value="320" x="-175.26" y="-35.56" smashed="yes">
+<attribute name="NAME" x="-177.8" y="-34.2646" size="0.9906" layer="25" ratio="10"/>
+<attribute name="POPULARITY" value="48" x="-175.26" y="-35.56" size="1.778" layer="27" display="off"/>
+<attribute name="SPICEPREFIX" value="R" x="-175.26" y="-35.56" size="1.778" layer="27" display="off"/>
+<attribute name="VALUE" x="-176.8856" y="-36.0426" size="0.9906" layer="27" ratio="10"/>
+</element>
 </elements>
 <signals>
-<signal name="+3.3V">
-<contactref element="U1" pad="J1_1"/>
-</signal>
 <signal name="+VBUS">
 <contactref element="U1" pad="J3_1"/>
@@
 <contactref element="X3" pad="3"/>
 <contactref element="U$1" pad="P$2"/>
-<contactref element="U2" pad="4"/>
 <contactref element="X1" pad="5"/>
 <contactref element="X1" pad="1"/>
+<contactref element="R5" pad="1"/>
+<contactref element="R4" pad="1"/>
+<contactref element="R3" pad="1"/>
+<contactref element="R2" pad="1"/>
+<contactref element="U2" pad="4"/>
 <contactref element="U2" pad="2"/>
+<wire x1="-179.07" y1="-30.48" x2="-179.07" y2="-35.56" width="0" layer="19" extent="1-1"/>
+<wire x1="-179.07" y1="-25.4" x2="-179.07" y2="-30.48" width="0" layer="19" extent="1-1"/>
+<wire x1="-179.07" y1="-20.32" x2="-179.07" y2="-25.4" width="0" layer="19" extent="1-1"/>
+<wire x1="-113.03" y1="-5.08" x2="-179.07" y2="-20.32" width="0" layer="19" extent="1-1"/>
 <wire x1="-105.41" y1="-7.62" x2="-113.03" y2="-5.08" width="0" layer="19" extent="1-1"/>
 <wire x1="-96.52" y1="-6.35" x2="-105.41" y2="-7.62" width="0" layer="19" extent="1-1"/>
@@
 <signal name="UART_TX">
 <contactref element="X3" pad="1"/>
+<contactref element="U1" pad="J1_3"/>
+<wire x1="-62.23" y1="33.02" x2="-101.6" y2="-6.35" width="0" layer="19" extent="1-1"/>
 </signal>
 <signal name="UART_RX">
 <contactref element="X3" pad="2"/>
-</signal>
-<signal name="N$4">
-<contactref element="U$1" pad="P$5"/>
-</signal>
-<signal name="N$5">
-<contactref element="U$1" pad="P$3"/>
-</signal>
-<signal name="SCL">
-<contactref element="U$1" pad="P$1"/>
-</signal>
-<signal name="SDA">
-<contactref element="U$1" pad="P$6"/>
-</signal>
-<signal name="10V">
-<contactref element="SP1" pad="2"/>
+<contactref element="U1" pad="J1_4"/>
+<wire x1="-62.23" y1="30.48" x2="-99.06" y2="-6.35" width="0" layer="19" extent="1-1"/>
 </signal>
 <signal name="VCC">
 <contactref element="U$1" pad="P$4"/>
-</signal>
-<signal name="N$1">
-<contactref element="SP1" pad="1"/>
-<contactref element="U2" pad="5"/>
-<wire x1="-22.3012" y1="115.57" x2="-105.41" y2="-5.08" width="0" layer="19" extent="1-1"/>
+<contactref element="U1" pad="J1_1"/>
+<wire x1="-62.23" y1="38.1" x2="-39.6875" y2="114.3" width="0" layer="19" extent="1-1"/>
 </signal>
 <signal name="N$9">
@@
 <wire x1="-59.69" y1="17.78" x2="-52.96" y2="105.85" width="0" layer="19" extent="1-1"/>
 </signal>
+<signal name="N$16">
+<contactref element="U1" pad="J1_7"/>
+<contactref element="U$2" pad="5"/>
+<wire x1="-62.23" y1="22.86" x2="-145.1" y2="-11.43" width="0" layer="19" extent="1-1"/>
+</signal>
+<signal name="N$17">
+<contactref element="U1" pad="J1_2"/>
+<contactref element="U$2" pad="6"/>
+<wire x1="-62.23" y1="35.56" x2="-142.56" y2="-11.43" width="0" layer="19" extent="1-1"/>
+</signal>
+<signal name="N$18">
+<contactref element="U1" pad="J2_7"/>
+<contactref element="U$2" pad="7"/>
+<wire x1="-16.51" y1="22.86" x2="-140.02" y2="-11.43" width="0" layer="19" extent="1-1"/>
+</signal>
+<signal name="N$19">
+<contactref element="U1" pad="J2_6"/>
+<contactref element="U$2" pad="8"/>
+<wire x1="-16.51" y1="25.4" x2="-137.48" y2="-11.43" width="0" layer="19" extent="1-1"/>
+</signal>
+<signal name="N$20">
+<contactref element="U1" pad="J3_3"/>
+<contactref element="U$2" pad="1"/>
+<contactref element="R5" pad="2"/>
+<wire x1="-155.26" y1="-11.43" x2="-171.45" y2="-35.56" width="0" layer="19" extent="1-1"/>
+<wire x1="-59.69" y1="33.02" x2="-155.26" y2="-11.43" width="0" layer="19" extent="1-1"/>
+</signal>
+<signal name="N$14">
+<contactref element="R4" pad="2"/>
+<contactref element="U$2" pad="2"/>
+<contactref element="U1" pad="J3_4"/>
+<wire x1="-152.72" y1="-11.43" x2="-171.45" y2="-30.48" width="0" layer="19" extent="1-1"/>
+<wire x1="-59.69" y1="30.48" x2="-152.72" y2="-11.43" width="0" layer="19" extent="1-1"/>
+</signal>
+<signal name="N$3">
+<contactref element="U$2" pad="3"/>
+<contactref element="R3" pad="2"/>
+<contactref element="U1" pad="J3_5"/>
+<wire x1="-150.18" y1="-11.43" x2="-171.45" y2="-25.4" width="0" layer="19" extent="1-1"/>
+<wire x1="-59.69" y1="27.94" x2="-150.18" y2="-11.43" width="0" layer="19" extent="1-1"/>
+</signal>
+<signal name="N$13">
+<contactref element="U$2" pad="4"/>
+<contactref element="R2" pad="2"/>
+<contactref element="U1" pad="J3_6"/>
+<wire x1="-147.64" y1="-11.43" x2="-171.45" y2="-20.32" width="0" layer="19" extent="1-1"/>
+<wire x1="-59.69" y1="25.4" x2="-147.64" y2="-11.43" width="0" layer="19" extent="1-1"/>
+</signal>
+<signal name="N$4">
+<contactref element="U$1" pad="P$1"/>
+<contactref element="U1" pad="J1_6"/>
+<wire x1="-62.23" y1="25.4" x2="-41.5925" y2="111.76" width="0" layer="19" extent="1-1"/>
+</signal>
+<signal name="N$5">
+<contactref element="U1" pad="J1_5"/>
+<contactref element="U$1" pad="P$6"/>
+<wire x1="-62.23" y1="27.94" x2="-41.5925" y2="114.3" width="0" layer="19" extent="1-1"/>
+</signal>
+<signal name="N$12">
+<contactref element="U2" pad="5"/>
+<contactref element="SP1" pad="1"/>
+<wire x1="-22.3012" y1="115.57" x2="-105.41" y2="-5.08" width="0" layer="19" extent="1-1"/>
+</signal>
+<signal name="10V">
+<contactref element="SP1" pad="2"/>
+</signal>
+<signal name="N$1">
+<contactref element="U1" pad="J4_3"/>
+<contactref element="R1" pad="2"/>
+<wire x1="-19.05" y1="33.02" x2="-105.41" y2="-15.24" width="0" layer="19" extent="1-1"/>
+</signal>
 <signal name="N$11">
-<contactref element="R1" pad="2"/>
-<contactref element="U1" pad="J1_6"/>
-<wire x1="-62.23" y1="25.4" x2="-105.41" y2="-15.24" width="0" layer="19" extent="1-1"/>
-</signal>
-<signal name="N$12">
+<contactref element="U2" pad="1"/>
 <contactref element="R1" pad="1"/>
-<contactref element="U2" pad="1"/>
 <wire x1="-113.03" y1="-2.54" x2="-113.03" y2="-15.24" width="0" layer="19" extent="1-1"/>
 </signal>
+<signal name="VDD">
+<contactref element="X1" pad="2"/>
+</signal>
 </signals>

Commit message: final final schematic
Parts:
- added R6, R7: 8.2k, rcl:0204/7
- R1: value 320 -> 520
- R2, R3, R4, R5: value 320 -> 10k
Connections:
- net N$4: now also R6.1
- net N$5: now also R7.1
- net VCC: now also R6.2, R7.2
Changed lines of the file:
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@@
 <attribute name="VALUE" x="-112.22475" y="-10.338309375" size="1.272009375" layer="27"/>
 </element>
-<element name="R1" library="rcl" library_urn="urn:adsk.eagle:library:334" package="0204/7" package3d_urn="urn:adsk.eagle:package:23498/2" value="320" x="-109.22" y="-15.24" smashed="yes">
+<element name="R1" library="rcl" library_urn="urn:adsk.eagle:library:334" package="0204/7" package3d_urn="urn:adsk.eagle:package:23498/2" value="520" x="-109.22" y="-15.24" smashed="yes">
 <attribute name="NAME" x="-111.76" y="-13.9446" size="0.9906" layer="25" ratio="10"/>
 <attribute name="POPULARITY" value="48" x="-109.22" y="-15.24" size="1.778" layer="27" display="off"/>
@@
 <attribute name="VALUE" x="-128.1" y="-11.555" size="1.27" layer="27"/>
 </element>
-<element name="R2" library="rcl" library_urn="urn:adsk.eagle:library:334" package="0204/7" package3d_urn="urn:adsk.eagle:package:23498/2" value="320" x="-175.26" y="-20.32" smashed="yes">
+<element name="R2" library="rcl" library_urn="urn:adsk.eagle:library:334" package="0204/7" package3d_urn="urn:adsk.eagle:package:23498/2" value="10k" x="-175.26" y="-20.32" smashed="yes">
 <attribute name="NAME" x="-177.8" y="-19.0246" size="0.9906" layer="25" ratio="10"/>
 <attribute name="POPULARITY" value="48" x="-175.26" y="-20.32" size="1.778" layer="27" display="off"/>
@@
 <attribute name="VALUE" x="-176.8856" y="-20.8026" size="0.9906" layer="27" ratio="10"/>
 </element>
-<element name="R3" library="rcl" library_urn="urn:adsk.eagle:library:334" package="0204/7" package3d_urn="urn:adsk.eagle:package:23498/2" value="320" x="-175.26" y="-25.4" smashed="yes">
+<element name="R3" library="rcl" library_urn="urn:adsk.eagle:library:334" package="0204/7" package3d_urn="urn:adsk.eagle:package:23498/2" value="10k" x="-175.26" y="-25.4" smashed="yes">
 <attribute name="NAME" x="-177.8" y="-24.1046" size="0.9906" layer="25" ratio="10"/>
 <attribute name="POPULARITY" value="48" x="-175.26" y="-25.4" size="1.778" layer="27" display="off"/>
@@
 <attribute name="VALUE" x="-176.8856" y="-25.8826" size="0.9906" layer="27" ratio="10"/>
 </element>
-<element name="R4" library="rcl" library_urn="urn:adsk.eagle:library:334" package="0204/7" package3d_urn="urn:adsk.eagle:package:23498/2" value="320" x="-175.26" y="-30.48" smashed="yes">
+<element name="R4" library="rcl" library_urn="urn:adsk.eagle:library:334" package="0204/7" package3d_urn="urn:adsk.eagle:package:23498/2" value="10k" x="-175.26" y="-30.48" smashed="yes">
 <attribute name="NAME" x="-177.8" y="-29.1846" size="0.9906" layer="25" ratio="10"/>
 <attribute name="POPULARITY" value="48" x="-175.26" y="-30.48" size="1.778" layer="27" display="off"/>
@@
 <attribute name="VALUE" x="-176.8856" y="-30.9626" size="0.9906" layer="27" ratio="10"/>
 </element>
-<element name="R5" library="rcl" library_urn="urn:adsk.eagle:library:334" package="0204/7" package3d_urn="urn:adsk.eagle:package:23498/2" value="320" x="-175.26" y="-35.56" smashed="yes">
+<element name="R5" library="rcl" library_urn="urn:adsk.eagle:library:334" package="0204/7" package3d_urn="urn:adsk.eagle:package:23498/2" value="10k" x="-175.26" y="-35.56" smashed="yes">
 <attribute name="NAME" x="-177.8" y="-34.2646" size="0.9906" layer="25" ratio="10"/>
 <attribute name="POPULARITY" value="48" x="-175.26" y="-35.56" size="1.778" layer="27" display="off"/>
 <attribute name="SPICEPREFIX" value="R" x="-175.26" y="-35.56" size="1.778" layer="27" display="off"/>
 <attribute name="VALUE" x="-176.8856" y="-36.0426" size="0.9906" layer="27" ratio="10"/>
+</element>
+<element name="R6" library="rcl" library_urn="urn:adsk.eagle:library:334" package="0204/7" package3d_urn="urn:adsk.eagle:package:23498/2" value="8.2k" x="-175.26" y="-40.64" smashed="yes">
+<attribute name="NAME" x="-177.8" y="-39.3446" size="0.9906" layer="25" ratio="10"/>
+<attribute name="POPULARITY" value="48" x="-175.26" y="-40.64" size="1.778" layer="27" display="off"/>
+<attribute name="SPICEPREFIX" value="R" x="-175.26" y="-40.64" size="1.778" layer="27" display="off"/>
+<attribute name="VALUE" x="-176.8856" y="-41.1226" size="0.9906" layer="27" ratio="10"/>
+</element>
+<element name="R7" library="rcl" library_urn="urn:adsk.eagle:library:334" package="0204/7" package3d_urn="urn:adsk.eagle:package:23498/2" value="8.2k" x="-175.26" y="-45.72" smashed="yes">
+<attribute name="NAME" x="-177.8" y="-44.4246" size="0.9906" layer="25" ratio="10"/>
+<attribute name="POPULARITY" value="48" x="-175.26" y="-45.72" size="1.778" layer="27" display="off"/>
+<attribute name="SPICEPREFIX" value="R" x="-175.26" y="-45.72" size="1.778" layer="27" display="off"/>
+<attribute name="VALUE" x="-176.8856" y="-46.2026" size="0.9906" layer="27" ratio="10"/>
 </element>
 </elements>
@@
 <contactref element="U$1" pad="P$4"/>
 <contactref element="U1" pad="J1_1"/>
-<wire x1="-62.23" y1="38.1" x2="-39.6875" y2="114.3" width="0" layer="19" extent="1-1"/>
+<contactref element="R6" pad="2"/>
+<contactref element="R7" pad="2"/>
+<wire x1="-171.45" y1="-40.64" x2="-171.45" y2="-45.72" width="0" layer="19" extent="1-1"/>
+<wire x1="-62.23" y1="38.1" x2="-171.45" y2="-40.64" width="0" layer="19" extent="1-1"/>
+<wire x1="-39.6875" y1="114.3" x2="-62.23" y2="38.1" width="0" layer="19" extent="1-1"/>
 </signal>
 <signal name="N$9">
@@
 <contactref element="U$1" pad="P$1"/>
 <contactref element="U1" pad="J1_6"/>
-<wire x1="-62.23" y1="25.4" x2="-41.5925" y2="111.76" width="0" layer="19" extent="1-1"/>
+<contactref element="R6" pad="1"/>
+<wire x1="-62.23" y1="25.4" x2="-179.07" y2="-40.64" width="0" layer="19" extent="1-1"/>
+<wire x1="-41.5925" y1="111.76" x2="-62.23" y2="25.4" width="0" layer="19" extent="1-1"/>
 </signal>
 <signal name="N$5">
 <contactref element="U1" pad="J1_5"/>
 <contactref element="U$1" pad="P$6"/>
-<wire x1="-62.23" y1="27.94" x2="-41.5925" y2="114.3" width="0" layer="19" extent="1-1"/>
+<contactref element="R7" pad="1"/>
+<wire x1="-62.23" y1="27.94" x2="-179.07" y2="-45.72" width="0" layer="19" extent="1-1"/>
+<wire x1="-41.5925" y1="114.3" x2="-62.23" y2="27.94" width="0" layer="19" extent="1-1"/>
 </signal>
 <signal name="N$12">
