File: PCB/Shematich_v1.brd (EAGLE design)
At the start: 100 x 80 mm, 14 parts, among them U1 EK-TM4C123GXL, U2 4N25, X1 HD44780LCD-1602, X3 22-23-2031

Commit message: final final final schematic (ready for hardware)
Connections:
- removed net +VBUS: U1.J3_1
- removed net N$5: R7.1, U$1.P$6, U1.J1_5
- new net N$21: R6.1, U$1.P$1, U1.J1_5
- net N$1: now also U1.J2_2; no longer U1.J4_3
- net N$13: now also U1.J4_8; no longer U1.J3_6
- net N$14: now also U1.J3_5; no longer U1.J3_4
- net N$16: now also U1.J4_3; no longer U1.J1_7
- net N$17: now also U1.J1_7; no longer U1.J1_2
- net N$18: now also U1.J1_2; no longer U1.J2_7
- net N$19: now also U1.J2_7; no longer U1.J2_6
- net N$20: now also U1.J3_4; no longer U1.J3_3
- net N$3: now also U1.J3_6; no longer U1.J3_5
- net N$4: now also R7.1, U$1.P$6; no longer R6.1, U$1.P$1
- net VDD: now also U1.J3_1
Changed lines of the file:
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@@
 </elements>
 <signals>
-<signal name="+VBUS">
-<contactref element="U1" pad="J3_1"/>
-</signal>
 <signal name="GND">
 <contactref element="U1" pad="J2_1"/>
@@
 </signal>
 <signal name="N$16">
-<contactref element="U1" pad="J1_7"/>
 <contactref element="U$2" pad="5"/>
-<wire x1="-62.23" y1="22.86" x2="-145.1" y2="-11.43" width="0" layer="19" extent="1-1"/>
+<contactref element="U1" pad="J4_3"/>
+<wire x1="-19.05" y1="33.02" x2="-145.1" y2="-11.43" width="0" layer="19" extent="1-1"/>
 </signal>
 <signal name="N$17">
-<contactref element="U1" pad="J1_2"/>
 <contactref element="U$2" pad="6"/>
-<wire x1="-62.23" y1="35.56" x2="-142.56" y2="-11.43" width="0" layer="19" extent="1-1"/>
+<contactref element="U1" pad="J1_7"/>
+<wire x1="-62.23" y1="22.86" x2="-142.56" y2="-11.43" width="0" layer="19" extent="1-1"/>
 </signal>
 <signal name="N$18">
-<contactref element="U1" pad="J2_7"/>
 <contactref element="U$2" pad="7"/>
-<wire x1="-16.51" y1="22.86" x2="-140.02" y2="-11.43" width="0" layer="19" extent="1-1"/>
+<contactref element="U1" pad="J1_2"/>
+<wire x1="-62.23" y1="35.56" x2="-140.02" y2="-11.43" width="0" layer="19" extent="1-1"/>
 </signal>
 <signal name="N$19">
-<contactref element="U1" pad="J2_6"/>
 <contactref element="U$2" pad="8"/>
-<wire x1="-16.51" y1="25.4" x2="-137.48" y2="-11.43" width="0" layer="19" extent="1-1"/>
+<contactref element="U1" pad="J2_7"/>
+<wire x1="-16.51" y1="22.86" x2="-137.48" y2="-11.43" width="0" layer="19" extent="1-1"/>
 </signal>
 <signal name="N$20">
-<contactref element="U1" pad="J3_3"/>
 <contactref element="U$2" pad="1"/>
 <contactref element="R5" pad="2"/>
+<contactref element="U1" pad="J3_4"/>
 <wire x1="-155.26" y1="-11.43" x2="-171.45" y2="-35.56" width="0" layer="19" extent="1-1"/>
-<wire x1="-59.69" y1="33.02" x2="-155.26" y2="-11.43" width="0" layer="19" extent="1-1"/>
+<wire x1="-59.69" y1="30.48" x2="-155.26" y2="-11.43" width="0" layer="19" extent="1-1"/>
 </signal>
 <signal name="N$14">
 <contactref element="R4" pad="2"/>
 <contactref element="U$2" pad="2"/>
-<contactref element="U1" pad="J3_4"/>
+<contactref element="U1" pad="J3_5"/>
 <wire x1="-152.72" y1="-11.43" x2="-171.45" y2="-30.48" width="0" layer="19" extent="1-1"/>
-<wire x1="-59.69" y1="30.48" x2="-152.72" y2="-11.43" width="0" layer="19" extent="1-1"/>
+<wire x1="-59.69" y1="27.94" x2="-152.72" y2="-11.43" width="0" layer="19" extent="1-1"/>
 </signal>
 <signal name="N$3">
 <contactref element="U$2" pad="3"/>
 <contactref element="R3" pad="2"/>
-<contactref element="U1" pad="J3_5"/>
+<contactref element="U1" pad="J3_6"/>
 <wire x1="-150.18" y1="-11.43" x2="-171.45" y2="-25.4" width="0" layer="19" extent="1-1"/>
-<wire x1="-59.69" y1="27.94" x2="-150.18" y2="-11.43" width="0" layer="19" extent="1-1"/>
+<wire x1="-59.69" y1="25.4" x2="-150.18" y2="-11.43" width="0" layer="19" extent="1-1"/>
 </signal>
 <signal name="N$13">
 <contactref element="U$2" pad="4"/>
 <contactref element="R2" pad="2"/>
-<contactref element="U1" pad="J3_6"/>
+<contactref element="U1" pad="J4_8"/>
 <wire x1="-147.64" y1="-11.43" x2="-171.45" y2="-20.32" width="0" layer="19" extent="1-1"/>
-<wire x1="-59.69" y1="25.4" x2="-147.64" y2="-11.43" width="0" layer="19" extent="1-1"/>
+<wire x1="-19.05" y1="20.32" x2="-147.64" y2="-11.43" width="0" layer="19" extent="1-1"/>
 </signal>
 <signal name="N$4">
-<contactref element="U$1" pad="P$1"/>
 <contactref element="U1" pad="J1_6"/>
-<contactref element="R6" pad="1"/>
-<wire x1="-62.23" y1="25.4" x2="-179.07" y2="-40.64" width="0" layer="19" extent="1-1"/>
-<wire x1="-41.5925" y1="111.76" x2="-62.23" y2="25.4" width="0" layer="19" extent="1-1"/>
-</signal>
-<signal name="N$5">
-<contactref element="U1" pad="J1_5"/>
 <contactref element="U$1" pad="P$6"/>
 <contactref element="R7" pad="1"/>
-<wire x1="-62.23" y1="27.94" x2="-179.07" y2="-45.72" width="0" layer="19" extent="1-1"/>
-<wire x1="-41.5925" y1="114.3" x2="-62.23" y2="27.94" width="0" layer="19" extent="1-1"/>
+<wire x1="-62.23" y1="25.4" x2="-179.07" y2="-45.72" width="0" layer="19" extent="1-1"/>
+<wire x1="-41.5925" y1="114.3" x2="-62.23" y2="25.4" width="0" layer="19" extent="1-1"/>
 </signal>
 <signal name="N$12">
@@
 <contactref element="SP1" pad="2"/>
 </signal>
-<signal name="N$1">
-<contactref element="U1" pad="J4_3"/>
-<contactref element="R1" pad="2"/>
-<wire x1="-19.05" y1="33.02" x2="-105.41" y2="-15.24" width="0" layer="19" extent="1-1"/>
-</signal>
 <signal name="N$11">
 <contactref element="U2" pad="1"/>
@@
 <signal name="VDD">
 <contactref element="X1" pad="2"/>
+<contactref element="U1" pad="J3_1"/>
+<wire x1="-59.69" y1="38.1" x2="-83.44" y2="105.85" width="0" layer="19" extent="1-1"/>
+</signal>
+<signal name="N$1">
+<contactref element="U1" pad="J2_2"/>
+<contactref element="R1" pad="2"/>
+<wire x1="-16.51" y1="35.56" x2="-105.41" y2="-15.24" width="0" layer="19" extent="1-1"/>
+</signal>
+<signal name="N$21">
+<contactref element="U$1" pad="P$1"/>
+<contactref element="R6" pad="1"/>
+<contactref element="U1" pad="J1_5"/>
+<wire x1="-62.23" y1="27.94" x2="-179.07" y2="-40.64" width="0" layer="19" extent="1-1"/>
+<wire x1="-41.5925" y1="111.76" x2="-62.23" y2="27.94" width="0" layer="19" extent="1-1"/>
 </signal>
 </signals>

Commit message: schematic updated
Connections:
- net N$1: now also U1.J3_3; no longer U1.J2_2
- net N$12: now also U2.6
Changed lines of the file:
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@@
 <contactref element="U2" pad="5"/>
 <contactref element="SP1" pad="1"/>
-<wire x1="-22.3012" y1="115.57" x2="-105.41" y2="-5.08" width="0" layer="19" extent="1-1"/>
+<contactref element="U2" pad="6"/>
+<wire x1="-105.41" y1="-2.54" x2="-105.41" y2="-5.08" width="0" layer="19" extent="1-1"/>
+<wire x1="-22.3012" y1="115.57" x2="-105.41" y2="-2.54" width="0" layer="19" extent="1-1"/>
 </signal>
 <signal name="10V">
@@
 <wire x1="-59.69" y1="38.1" x2="-83.44" y2="105.85" width="0" layer="19" extent="1-1"/>
 </signal>
-<signal name="N$1">
-<contactref element="U1" pad="J2_2"/>
-<contactref element="R1" pad="2"/>
-<wire x1="-16.51" y1="35.56" x2="-105.41" y2="-15.24" width="0" layer="19" extent="1-1"/>
-</signal>
 <signal name="N$21">
 <contactref element="U$1" pad="P$1"/>
@@
 <wire x1="-41.5925" y1="111.76" x2="-62.23" y2="27.94" width="0" layer="19" extent="1-1"/>
 </signal>
+<signal name="N$1">
+<contactref element="R1" pad="2"/>
+<contactref element="U1" pad="J3_3"/>
+<wire x1="-59.69" y1="33.02" x2="-105.41" y2="-15.24" width="0" layer="19" extent="1-1"/>
+</signal>
 </signals>
