File: PCB/Shematich_v1.sch (EAGLE design)
At the start: 8 parts, among them U1 EK-TM4C123GXL, U2 4N25, X1 HD44780LCD-1602, X2 22-23-2081, X3 22-23-2031

Commit message: shematic 2
Parts:
- removed OK1: SFH618A-3, optocoupler:SFH618A-3
- added R1: 320, rcl:R-US_0204/7
Connections:
- net N$3 renamed 10V
- new net N$10: U1.PC6, X1.RS
- new net N$11: R1.2, U1.PE5
- new net N$12: R1.1, U2.A
- new net N$2: U1.PE0, X1.DB4
- new net N$6: U1.PE1, X1.DB5
- new net N$7: U1.PE2, X1.DB6
- new net N$8: U1.PE3, X1.DB7
- new net N$9: U1.PC7, X1.E
- net GND: now also U2.E, U2.K, X1.RW, X1.VSS; no longer OK1.C
- net N$1: now also U2.C; no longer OK1.A
Other:
- moved on the sheet: SP1, U1, U2, X1, X3-1, X3-2, X3-3

Commit message: shematic 3
Parts:
- added U$2: (no value), keypad_4x4_raw:KEYPAD4X4
Changed lines of the file:
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@@
 <part name="SUPPLY5" library="supply2" library_urn="urn:adsk.eagle:library:372" deviceset="GND" device=""/>
 <part name="R1" library="rcl" library_urn="urn:adsk.eagle:library:334" deviceset="R-US_" device="0204/7" package3d_urn="urn:adsk.eagle:package:23498/2" value="320"/>
+<part name="U$2" library="keypad_4x4_raw" deviceset="KEYPAD4X4" device=""/>
 </parts>
 <sheets>
@@
 <attribute name="VALUE" x="36.322" y="1.27" size="1.778" layer="96" rot="R90"/>
 </instance>
+<instance part="U$2" gate="G$1" x="96.52" y="50.8" smashed="yes" rot="MR0">
+<attribute name="NAME" x="114.3" y="66.04" size="1.27" layer="95" rot="MR0"/>
+<attribute name="VALUE" x="106.68" y="66.04" size="1.27" layer="96" rot="MR0"/>
+</instance>
 </instances>

Commit message: final schematic
Parts:
- removed X2: 22-23-2081, con-molex:22-23-2081
- added R2, R3, R4, R5: 320, rcl:R-US_0204/7
Connections:
- removed net N$11 (its old number): R1.2, U1.PE5
- removed net SCL: U$1.SCL
- removed net SDA: U$1.SDA
- new net N$1: R1.2, U1.PB3
- new net N$13: R2.2, U$2.C4, U1.PD3
- new net N$14: R4.2, U$2.C2, U1.PD1
- new net N$16: U$2.R1, U1.PB4
- new net N$17: U$2.R2, U1.PB5
- new net N$18: U$2.R3, U1.PB6
- new net N$19: U$2.R4, U1.PB7
- new net N$20: R5.2, U$2.C1, U1.PD0
- new net N$3: R3.2, U$2.C3, U1.PD2
- new net VDD: X1.VDD
- net GND: now also R2.1, R3.1, R4.1, R5.1, U1.GND
- net N$4: now also U$1.SCL, U1.PE5; no longer U$1.ADR0
- net N$5: now also U$1.SDA, U1.PE4; no longer U$1.ADR1
- net UART_RX: now also U1.PB1
- net UART_TX: now also U1.PB0
- net VCC: now also U1.+3.3V
Other:
- moved on the sheet: R1, SP1, U2, X3-1, X3-2, X3-3

Commit message: final final schematic
Parts:
- added R6, R7: 8.2k, rcl:R-US_0204/7
- R1: value 320 -> 520
- R2, R3, R4, R5: value 320 -> 10k
Connections:
- net N$4: now also R6.1
- net N$5: now also R7.1
- net VCC: now also R6.2, R7.2
Changed lines of the file:
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@@
 <part name="U2" library="4N25" deviceset="4N25" device=""/>
 <part name="SUPPLY5" library="supply2" library_urn="urn:adsk.eagle:library:372" deviceset="GND" device=""/>
-<part name="R1" library="rcl" library_urn="urn:adsk.eagle:library:334" deviceset="R-US_" device="0204/7" package3d_urn="urn:adsk.eagle:package:23498/2" value="320"/>
+<part name="R1" library="rcl" library_urn="urn:adsk.eagle:library:334" deviceset="R-US_" device="0204/7" package3d_urn="urn:adsk.eagle:package:23498/2" value="520"/>
 <part name="U$2" library="keypad_4x4_raw" deviceset="KEYPAD4X4" device=""/>
-<part name="R2" library="rcl" library_urn="urn:adsk.eagle:library:334" deviceset="R-US_" device="0204/7" package3d_urn="urn:adsk.eagle:package:23498/2" value="320"/>
-<part name="R3" library="rcl" library_urn="urn:adsk.eagle:library:334" deviceset="R-US_" device="0204/7" package3d_urn="urn:adsk.eagle:package:23498/2" value="320"/>
-<part name="R4" library="rcl" library_urn="urn:adsk.eagle:library:334" deviceset="R-US_" device="0204/7" package3d_urn="urn:adsk.eagle:package:23498/2" value="320"/>
-<part name="R5" library="rcl" library_urn="urn:adsk.eagle:library:334" deviceset="R-US_" device="0204/7" package3d_urn="urn:adsk.eagle:package:23498/2" value="320"/>
+<part name="R2" library="rcl" library_urn="urn:adsk.eagle:library:334" deviceset="R-US_" device="0204/7" package3d_urn="urn:adsk.eagle:package:23498/2" value="10k"/>
+<part name="R3" library="rcl" library_urn="urn:adsk.eagle:library:334" deviceset="R-US_" device="0204/7" package3d_urn="urn:adsk.eagle:package:23498/2" value="10k"/>
+<part name="R4" library="rcl" library_urn="urn:adsk.eagle:library:334" deviceset="R-US_" device="0204/7" package3d_urn="urn:adsk.eagle:package:23498/2" value="10k"/>
+<part name="R5" library="rcl" library_urn="urn:adsk.eagle:library:334" deviceset="R-US_" device="0204/7" package3d_urn="urn:adsk.eagle:package:23498/2" value="10k"/>
 <part name="SUPPLY6" library="supply2" library_urn="urn:adsk.eagle:library:372" deviceset="GND" device=""/>
 <part name="SUPPLY7" library="supply2" library_urn="urn:adsk.eagle:library:372" deviceset="GND" device=""/>
@@
 <part name="SUPPLY11" library="supply2" library_urn="urn:adsk.eagle:library:372" deviceset="VCC" device=""/>
 <part name="SUPPLY12" library="supply2" library_urn="urn:adsk.eagle:library:372" deviceset="VCC" device=""/>
+<part name="R6" library="rcl" library_urn="urn:adsk.eagle:library:334" deviceset="R-US_" device="0204/7" package3d_urn="urn:adsk.eagle:package:23498/2" value="8.2k"/>
+<part name="SUPPLY13" library="supply2" library_urn="urn:adsk.eagle:library:372" deviceset="VCC" device=""/>
+<part name="R7" library="rcl" library_urn="urn:adsk.eagle:library:334" deviceset="R-US_" device="0204/7" package3d_urn="urn:adsk.eagle:package:23498/2" value="8.2k"/>
+<part name="SUPPLY14" library="supply2" library_urn="urn:adsk.eagle:library:372" deviceset="VCC" device=""/>
 </parts>
 <sheets>
@@
 <attribute name="VALUE" x="78.105" y="106.045" size="1.778" layer="96"/>
 </instance>
+<instance part="R6" gate="G$1" x="25.4" y="13.97" smashed="yes" rot="R90">
+<attribute name="NAME" x="23.9014" y="10.16" size="1.778" layer="95" rot="R90"/>
+<attribute name="VALUE" x="28.702" y="10.16" size="1.778" layer="96" rot="R90"/>
+</instance>
+<instance part="SUPPLY13" gate="G$1" x="25.4" y="21.59" smashed="yes">
+<attribute name="VALUE" x="23.495" y="24.765" size="1.778" layer="96"/>
+</instance>
+<instance part="R7" gate="G$1" x="33.02" y="6.35" smashed="yes" rot="R90">
+<attribute name="NAME" x="31.5214" y="2.54" size="1.778" layer="95" rot="R90"/>
+<attribute name="VALUE" x="36.322" y="2.54" size="1.778" layer="96" rot="R90"/>
+</instance>
+<instance part="SUPPLY14" gate="G$1" x="33.02" y="13.97" smashed="yes">
+<attribute name="VALUE" x="31.115" y="17.145" size="1.778" layer="96"/>
+</instance>
 </instances>
 <busses>
@@
 <pinref part="SUPPLY12" gate="G$1" pin="VCC"/>
 <wire x1="80.01" y1="96.52" x2="80.01" y2="100.33" width="0.1524" layer="91"/>
+</segment>
+<segment>
+<pinref part="SUPPLY13" gate="G$1" pin="VCC"/>
+<pinref part="R6" gate="G$1" pin="2"/>
+</segment>
+<segment>
+<pinref part="SUPPLY14" gate="G$1" pin="VCC"/>
+<pinref part="R7" gate="G$1" pin="2"/>
 </segment>
 </net>
@@
 <pinref part="U$1" gate="G$1" pin="SCL"/>
 <pinref part="U1" gate="G$1" pin="PE5"/>
-<wire x1="20.32" y1="8.89" x2="44.45" y2="8.89" width="0.1524" layer="91"/>
+<wire x1="20.32" y1="8.89" x2="25.4" y2="8.89" width="0.1524" layer="91"/>
+<wire x1="25.4" y1="8.89" x2="44.45" y2="8.89" width="0.1524" layer="91"/>
 <wire x1="44.45" y1="8.89" x2="44.45" y2="40.64" width="0.1524" layer="91"/>
+<pinref part="R6" gate="G$1" pin="1"/>
+<junction x="25.4" y="8.89"/>
 </segment>
 </net>
@@
 <pinref part="U$1" gate="G$1" pin="SDA"/>
 <wire x1="39.37" y1="43.18" x2="39.37" y2="1.27" width="0.1524" layer="91"/>
-<wire x1="39.37" y1="1.27" x2="20.32" y2="1.27" width="0.1524" layer="91"/>
-</segment>
-</net>
+<wire x1="39.37" y1="1.27" x2="33.02" y2="1.27" width="0.1524" layer="91"/>
+<pinref part="R7" gate="G$1" pin="1"/>
+<wire x1="33.02" y1="1.27" x2="20.32" y2="1.27" width="0.1524" layer="91"/>
+<junction x="33.02" y="1.27"/>
+</segment>
+</net>

Commit message: final final final schematic (ready for hardware)
Connections:
- removed net N$5: R7.1, U$1.SDA, U1.PE4
- new net N$21: R6.1, U$1.SCL, U1.PE4
- net N$1: now also U1.PB2; no longer U1.PB3
- net N$13: now also U1.PD6; no longer U1.PD3
- net N$14: now also U1.PD2; no longer U1.PD1
- net N$16: now also U1.PB3; no longer U1.PB4
- net N$17: now also U1.PB4; no longer U1.PB5
- net N$18: now also U1.PB5; no longer U1.PB6
- net N$19: now also U1.PB6; no longer U1.PB7
- net N$20: now also U1.PD1; no longer U1.PD0
- net N$3: now also U1.PD3; no longer U1.PD2
- net N$4: now also R7.1, U$1.SDA; no longer R6.1, U$1.SCL
- net VDD: now also U1.+VBUS

Commit message: schematic updated
Connections:
- net N$1: now also U1.PD0; no longer U1.PB2
- net N$12: now also U2.B
Other:
- moved on the sheet: R1, U2
Changed lines of the file:
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@@
 <attribute name="VALUE" x="-6.35" y="64.77" size="2.1844" layer="96" font="vector" rot="R270"/>
 </instance>
-<instance part="SUPPLY1" gate="GND" x="99.06" y="67.31" smashed="yes">
-<attribute name="VALUE" x="97.155" y="64.135" size="1.778" layer="96"/>
+<instance part="SUPPLY1" gate="GND" x="104.14" y="76.2" smashed="yes">
+<attribute name="VALUE" x="102.235" y="73.025" size="1.778" layer="96"/>
 </instance>
 <instance part="X3" gate="-1" x="107.95" y="116.84" smashed="yes">
@@
 <attribute name="VALUE" x="5.715" y="26.035" size="1.778" layer="96"/>
 </instance>
-<instance part="U2" gate="G$1" x="116.84" y="83.82" smashed="yes">
-<attribute name="NAME" x="104.1353" y="93.9838" size="2.540940625" layer="95"/>
-<attribute name="VALUE" x="104.1196" y="71.0996" size="2.54408125" layer="96"/>
+<instance part="U2" gate="G$1" x="121.92" y="83.82" smashed="yes">
+<attribute name="NAME" x="109.2153" y="93.9838" size="2.540940625" layer="95"/>
+<attribute name="VALUE" x="110.4696" y="69.8296" size="2.54408125" layer="96"/>
 </instance>
 <instance part="SUPPLY5" gate="GND" x="35.56" y="86.36" smashed="yes">
 <attribute name="VALUE" x="33.655" y="83.185" size="1.778" layer="96"/>
 </instance>
-<instance part="R1" gate="G$1" x="93.98" y="86.36" smashed="yes" rot="R270">
-<attribute name="NAME" x="95.4786" y="90.17" size="1.778" layer="95" rot="R270"/>
-<attribute name="VALUE" x="90.678" y="90.17" size="1.778" layer="96" rot="R270"/>
+<instance part="R1" gate="G$1" x="100.33" y="86.36" smashed="yes" rot="R270">
+<attribute name="NAME" x="101.8286" y="90.17" size="1.778" layer="95" rot="R270"/>
+<attribute name="VALUE" x="97.028" y="90.17" size="1.778" layer="96" rot="R270"/>
 </instance>
 <instance part="U$2" gate="G$1" x="96.52" y="50.8" smashed="yes" rot="MR0">
-<attribute name="NAME" x="100.33" y="67.31" size="1.27" layer="95" rot="MR0"/>
+<attribute name="NAME" x="96.52" y="50.8" size="1.27" layer="95" rot="MR0"/>
 <attribute name="VALUE" x="106.68" y="66.04" size="1.27" layer="96" rot="MR0"/>
 </instance>
@@
 <attribute name="VALUE" x="31.115" y="17.145" size="1.778" layer="96"/>
 </instance>
-<instance part="SUPPLY11" gate="GND" x="134.62" y="67.31" smashed="yes">
-<attribute name="VALUE" x="132.715" y="64.135" size="1.778" layer="96"/>
+<instance part="SUPPLY11" gate="GND" x="139.7" y="67.31" smashed="yes">
+<attribute name="VALUE" x="137.795" y="64.135" size="1.778" layer="96"/>
 </instance>
 </instances>
@@
 <segment>
 <pinref part="U2" gate="G$1" pin="E"/>
-<wire x1="134.62" y1="76.2" x2="134.62" y2="69.85" width="0.1524" layer="91"/>
+<wire x1="139.7" y1="76.2" x2="139.7" y2="69.85" width="0.1524" layer="91"/>
 <pinref part="SUPPLY11" gate="GND" pin="GND"/>
 </segment>
 <segment>
 <pinref part="U2" gate="G$1" pin="K"/>
-<wire x1="99.06" y1="83.82" x2="99.06" y2="69.85" width="0.1524" layer="91"/>
+<wire x1="104.14" y1="83.82" x2="104.14" y2="78.74" width="0.1524" layer="91"/>
 <pinref part="SUPPLY1" gate="GND" pin="GND"/>
 </segment>
@@
 <segment>
 <pinref part="U2" gate="G$1" pin="C"/>
-<wire x1="134.62" y1="83.82" x2="139.7" y2="83.82" width="0.1524" layer="91"/>
 <pinref part="SP1" gate="G$1" pin="1"/>
-<wire x1="139.7" y1="83.82" x2="139.7" y2="95.25" width="0.1524" layer="91"/>
+<wire x1="139.7" y1="83.82" x2="139.7" y2="91.44" width="0.1524" layer="91"/>
+<pinref part="U2" gate="G$1" pin="B"/>
+<wire x1="139.7" y1="91.44" x2="139.7" y2="95.25" width="0.1524" layer="91"/>
+<junction x="139.7" y="91.44"/>
 </segment>
 </net>
@@
 <pinref part="U2" gate="G$1" pin="A"/>
 <pinref part="R1" gate="G$1" pin="1"/>
-<wire x1="99.06" y1="91.44" x2="93.98" y2="91.44" width="0.1524" layer="91"/>
+<wire x1="104.14" y1="91.44" x2="100.33" y2="91.44" width="0.1524" layer="91"/>
 </segment>
 </net>
@@
 <wire x1="86.36" y1="101.6" x2="25.4" y2="101.6" width="0.1524" layer="91"/>
 <wire x1="25.4" y1="101.6" x2="25.4" y2="74.93" width="0.1524" layer="91"/>
-</segment>
-</net>
-<net name="N$1" class="0">
-<segment>
-<pinref part="U1" gate="G$1" pin="PB2"/>
-<wire x1="80.01" y1="83.82" x2="92.71" y2="83.82" width="0.1524" layer="91"/>
-<pinref part="R1" gate="G$1" pin="2"/>
-<wire x1="92.71" y1="83.82" x2="92.71" y2="81.28" width="0.1524" layer="91"/>
-<wire x1="92.71" y1="81.28" x2="93.98" y2="81.28" width="0.1524" layer="91"/>
 </segment>
 </net>
@@
 </segment>
 </net>
+<net name="N$1" class="0">
+<segment>
+<pinref part="R1" gate="G$1" pin="2"/>
+<pinref part="U1" gate="G$1" pin="PD0"/>
+<wire x1="100.33" y1="81.28" x2="100.33" y2="66.04" width="0.1524" layer="91"/>
+<wire x1="100.33" y1="66.04" x2="80.01" y2="66.04" width="0.1524" layer="91"/>
+</segment>
+</net>
